Commit message: Add

File: manip_teaching/urdf/camera_with_pump.urdf (robot description, URDF)
Before this commit: robot camera_with_pump2, 4 links, 3 joints
Links:
- link base_link: mass 0.395757124911999 -> 0.395757124912
- link t265_link: mass 0.0153522629829022 -> 0.0153522629828604
Joints:
- removed joint base_to_suction_joint
- removed joint base_to_t265_joint
- added joint t265_to_base_joint: type fixed, parent t265_link, child base_link, origin xyz=-0.0369126817859819 -0.0136161902876692 -0.0309999999999998 rpy=1.5707963267949 -0.0 1.5707963267949, axis 0. 0. 0., limit effort=0.0 velocity=0.0
- added joint t265_to_suction_frame_joint: type fixed, parent t265_link, child suction_frame, origin xyz=-0.03495 0.086636241608402 -0.047 rpy=0.0 -0.0 1.5707963267949, axis 0. 0. 0., limit effort=0.0 velocity=0.0
- joint base_to_d405_link: origin xyz=0.0827524318960711 0.0309999999999999 -0.0070373182140181 rpy=-1.5707963267949 -0.0 0.0 -> xyz=-0.04395 0.0691362416084019 0.0 rpy=0.0 -0.0 1.5707963267949; parent base_link -> t265_link
